File: tuxkeychain.kicad_pcb (KiCad board)
At the start: 6 copper layers, 45 x 25 mm, 45 parts, among them J1 Amphenol_10104111, Q2 2N7002, SW1 B3U-1000P, U1 JW5211, U2 JW5211, U3 JW5211, U4 F1C100s, U6 W25Q128JVS, Y1 24MHz

Commit message: rev 2
Parts:
- removed C1, C2: 2u2, Capacitor_SMD:C_0603_1608Metric
- removed C10, C11, C9: 22u, Capacitor_SMD:C_0603_1608Metric
- removed L1, L2, L3: 2u2, Inductor_SMD:L_0805_2012Metric
- removed R1, R2: 11k, Resistor_SMD:R_0603_1608Metric
- removed R3: 10k, Resistor_SMD:R_0603_1608Metric
- removed R4: 49k9, Resistor_SMD:R_0603_1608Metric
- removed R5: 36k, Resistor_SMD:R_0603_1608Metric
- removed R6: 8k2, Resistor_SMD:R_0603_1608Metric
- removed U1, U2, U3: JW5211, Package_TO_SOT_SMD:SOT-23-5
- added ?: , Graphics, F.Cu at (138.5, 51.7)
- added ? (x4): , Graphics, B.Cu at (138.5, 51.7)
- added ?: , DrillHole, B.Cu at (113.3, 56.8)
- added C19: 2u2, Capacitor_SMD:C_0603_1608Metric, F.Cu at (99.1, 102.0)
- added C20: 22u, Resistor_SMD:R_0603_1608Metric, F.Cu at (99.1, 94.0)
- added C21: 2u2, Capacitor_SMD:C_0603_1608Metric, F.Cu at (106.1, 102.0)
- added C22: 22u, Resistor_SMD:R_0603_1608Metric, F.Cu at (106.1, 94.0)
- added C23: 2u2, Capacitor_SMD:C_0603_1608Metric, F.Cu at (102.6, 102.0)
- added C24: 22u, Resistor_SMD:R_0603_1608Metric, F.Cu at (102.6, 94.0)
- added R13: 150k, Resistor_SMD:R_0603_1608Metric, F.Cu at (99.1, 95.5)
- added R14: 470k, Resistor_SMD:R_0603_1608Metric, F.Cu at (99.1, 97.0)
- added R15: 150k, Resistor_SMD:R_0603_1608Metric, F.Cu at (106.1, 95.5)
- added R16: 56k, Resistor_SMD:R_0603_1608Metric, F.Cu at (106.1, 97.0)
- added R17: 150k, Resistor_SMD:R_0603_1608Metric, F.Cu at (102.6, 95.5)
- added R18: 330k, Resistor_SMD:R_0603_1608Metric, F.Cu at (102.6, 97.0)
- added U5: TLV76701DRVx, Package_SON:WSON-6-1EP_2x2mm_P0.65mm_EP1x1.6mm, F.Cu at (99.2, 99.6)
- added U7: TLV76701DRVx, Package_SON:WSON-6-1EP_2x2mm_P0.65mm_EP1x1.6mm, F.Cu at (106.2, 99.6)
- added U8: TLV76701DRVx, Package_SON:WSON-6-1EP_2x2mm_P0.65mm_EP1x1.6mm, F.Cu at (102.7, 99.6)
- moved JP1 63.7 mm to (120.5, 104.6), turned to -90 degrees
- moved J1 59.5 mm to (113.3, 105.2), turned to 0 degrees
- moved U4 38.1 mm to (109.4, 81.8), turned to -135 degrees
- moved C18 37.2 mm to (48.5, 75.7), turned to 0 degrees
- moved R9 37.2 mm to (78.7, 134.7), turned to 0 degrees
- moved SW1 35.8 mm to (85.2, 119.5), turned to 0 degrees
- moved D1 33.5 mm to (67.5, 131.1)
- moved C17 32.4 mm to (48.5, 73.2), turned to 0 degrees
- moved R11 30.0 mm to (63.5, 128.9), turned to 0 degrees
- moved U6 29.9 mm to (81.8, 130.0), turned to 0 degrees
- moved R10 26.3 mm to (63.5, 126.4), turned to 0 degrees
- moved Q2 26.1 mm to (68.0, 127.6), turned to 0 degrees
- moved C6 25.6 mm to (63.6, 110.5), turned to 0 degrees
- moved R12 24.1 mm to (75.3, 120.2), turned to 0 degrees
- moved C5 24.1 mm to (63.6, 108.0), turned to 0 degrees
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Routing:
- net +3V3: track 93.5 -> 7.27 mm, vias 8 -> 1
- net +1V1: track 58.1 -> 7.27 mm, vias 4 -> 1
- net +2V6: track 52.8 -> 7.27 mm, vias 3 -> 1
- net GND: track 36.7 -> 0.00 mm, vias 7 -> 0
- net VBUS: track 42.1 -> 6.53 mm, vias 2 -> 0
- net SPI_CS: track 26.6 -> 0.00 mm, vias 2 -> 0
- net SPI_MISO: track 22.5 -> 0.00 mm, vias 2 -> 0
- net ~{RESET}: track 20.3 -> 0.00 mm, vias 2 -> 0
- net D-: track 15.7 -> 0.00 mm
- net D+: track 15.3 -> 0.00 mm
- net SPI_MOSI: track 14.7 -> 0.00 mm, vias 2 -> 0
- net SPI_CLK: track 13.8 -> 0.00 mm, vias 2 -> 0
- net STATUS: track 13.0 -> 0.00 mm, vias 2 -> 0
- net +5V: track 22.4 -> 12.1 mm
- net Net-(U4B-SVREF): track 9.33 -> 0.00 mm
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- removed copper zone on B.Cu, net GND
Other:
- board size 45 x 25 mm -> 50 x 60 mm
- board text added: "Rev. ${REVISION}"
- board text added: "Tux is 60x50mm"
- board text added: "allthingslinux.org"
- board text removed: "Tux Keychain Prototype Rev. ${REVISION}"

Commit message: imrptoravnemtn
Parts:
- added J2: JUSHUO AFC07-S24FCA-00, Connector_FFC-FPC:Jushuo_AFC07-S24FCA-00_1x24-1MP_P0.50_Horizontal, F.Cu at (112.0, 72.7)
- moved R11 76.8 mm to (72.6, 52.7)
- moved D1 72.6 mm to (68.5, 58.5)
- moved R10 72.6 mm to (64.5, 53.8)
- moved Q2 72.6 mm to (68.9, 55.0)
- moved C17 56.8 mm to (102.5, 90.7), turned to -135 degrees
- moved C3 56.0 mm to (115.0, 80.7), turned to 45 degrees
- moved C18 51.2 mm to (98.5, 86.7), turned to 45 degrees
- moved R12 50.6 mm to (115.8, 89.8), turned to -45 degrees
- moved SW1 39.9 mm to (114.5, 92.3), turned to -45 degrees
- moved C4 34.1 mm to (79.2, 75.2)
- moved C5 34.1 mm to (79.2, 77.7)
- moved C6 34.1 mm to (79.2, 80.2)
- moved C7 34.1 mm to (79.2, 82.7)
- moved U6 7.67 mm to (87.5, 135.2)
- moved U4 2.70 mm to (107.9, 84.0)
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Connections:
- U4 pad 1: unconnected-(U4A-HPL-Pad1) -> HPL
- U4 pad 3: unconnected-(U4A-HPCOM-Pad3) -> HPCOM
- U4 pad 39: unconnected-(U4A-PE10/CSI_D7/UART2_CTS/SPI1_MISO/EINTE10-Pad39) -> SPI1_MISO
- U4 pad 40: unconnected-(U4A-PE9/CSI_D6/UART2_RTS/SPI1_CLK/EINTE9-Pad40) -> SPI1_CLK
- U4 pad 41: unconnected-(U4A-PE8/CSI_D5/UART2_RX/SPI1_MOSI/EINTE8-Pad41) -> SPI1_MOSI
- U4 pad 42: unconnected-(U4A-PE7/CSI_D4/UART2_TX/SPI1_CS/EINTE7-Pad42) -> SPI1_CS
- U4 pad 53: JTAG_TCK -> SDC0_D2/JTAG_TCK
- U4 pad 54: unconnected-(U4A-PF4/SDC0_D3/UART0_TX/EINTF4-Pad54) -> SDC0_D3
- U4 pad 55: JTAG_TDO -> SDC0_CMD/JTAG_TDO
- U4 pad 56: unconnected-(U4A-PF2/SDC0_CLK/UART0_RX/EINTF2-Pad56) -> SDC0_CLK
- U4 pad 57: JTAG_TDI -> SDC0_D0/JTAG_TDI
- U4 pad 58: JTAG_TMS -> SDC0_D1/JTAG_TMS
- U4 pad 72: unconnected-(U4A-TVOUT-Pad72) -> TVOUT
- U4 pad 87: GND -> MICIN
- U4 pad 88: unconnected-(U4A-HPR-Pad88) -> HPR
Routing:
- net D+: track 0.00 -> 14.5 mm
- net D-: track 0.00 -> 14.1 mm
- net ~{RESET}: track 0.00 -> 7.34 mm
- net /CLKN: track 0.00 -> 7.34 mm
- net /CLKP: track 0.00 -> 4.78 mm
- net GND: track 0.00 -> 3.49 mm
- net +3V3: track 7.27 -> 9.40 mm

Commit message: Added expansion connectors to pcb
Parts:
- removed J2: JUSHUO AFC07-S24FCA-00, Connector_FFC-FPC:Jushuo_AFC07-S24FCA-00_1x24-1MP_P0.50_Horizontal
- added J3: EXPANSION, tuxkeychain:FFC_1x15_P0.5mm, F.Cu at (112.5, 72.2)
- added J5: Solder Pads, Connector_PinHeader_1.00mm:PinHeader_1x12_P1.00mm_Vertical_SMD_Pin1Left, F.Cu at (122.1, 89.2)
- moved R10 63.0 mm to (121.5, 80.7), turned to -90 degrees
- moved Q2 55.4 mm to (119.2, 78.2)
- moved D1 55.4 mm to (118.8, 81.7), turned to 180 degrees
- moved R11 49.4 mm to (115.5, 77.2), turned to 180 degrees
- moved R9 49.0 mm to (109.0, 96.2), turned to -90 degrees
- moved U6 46.1 mm to (115.0, 98.2)
- moved R8 43.0 mm to (102.6, 78.2), turned to 90 degrees
- moved C4 11.0 mm to (71.2, 82.7)
- moved C5 11.0 mm to (71.2, 85.2)
- moved C6 11.0 mm to (71.2, 87.7)
- moved C7 11.0 mm to (71.2, 90.2)

Commit message: work
Parts:
- C12, C13, C14, C15, C16, C17, C18, C19, C21, C23, C3, C4, C5, C6, C7, C8: footprint Capacitor_SMD:C_0603_1608Metric -> Capacitor_SMD:C_0402_1005Metric
- C20, C22, C24: footprint Resistor_SMD:R_0603_1608Metric -> Capacitor_SMD:C_0402_1005Metric
- J5: footprint Connector_PinHeader_1.00mm:PinHeader_1x12_P1.00mm_Vertical_SMD_Pin1Left -> tuxkeychain:SolderPads12
- R10, R11, R12, R13, R14, R15, R16, R17, R18, R7, R8, R9: footprint Resistor_SMD:R_0603_1608Metric -> Resistor_SMD:R_0402_1005Metric
- moved ? 73.3 mm to (65.6, 59.2), turned to 0 degrees
- moved ? 71.8 mm to (67.1, 59.2), turned to 0 degrees
- moved C3 71.2 mm to (44.4, 71.5), turned to 0 degrees
- moved ? 70.3 mm to (68.6, 59.2), turned to 0 degrees
- moved R10 63.0 mm to (58.6, 84.3), turned to 0 degrees
- moved SW1 61.5 mm to (61.9, 60.6), turned to 0 degrees
- moved D1 59.2 mm to (61.0, 68.6), turned to 0 degrees
- moved R12 55.1 mm to (61.5, 80.3), turned to 0 degrees
- moved Q2 54.1 mm to (66.7, 65.2)
- moved R11 54.0 mm to (61.5, 78.3), turned to 0 degrees
- moved R9 52.3 mm to (58.6, 82.3), turned to 0 degrees
- moved R8 44.0 mm to (58.6, 80.3), turned to 0 degrees
- moved C15 42.8 mm to (47.3, 75.4)
- moved C14 42.3 mm to (47.3, 73.4)
- moved C13 41.8 mm to (47.3, 71.5)
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Routing:
- net D+: track 14.5 -> 0.00 mm
- net D-: track 14.1 -> 0.00 mm
- net +5V: track 12.1 -> 24.2 mm, vias 0 -> 1
- net Net-(J1-Shield): track 11.0 -> 0.00 mm
- net SDC0_D2/JTAG_TCK: track 0.00 -> 8.57 mm
- net SDC0_D3: track 0.00 -> 8.53 mm
- net SDC0_CMD/JTAG_TDO: track 0.00 -> 8.49 mm
- net SDC0_CLK: track 0.00 -> 8.45 mm
- net SDC0_D0/JTAG_TDI: track 0.00 -> 8.40 mm
- net SDC0_D1/JTAG_TMS: track 0.00 -> 8.36 mm
- net ~{RESET}: track 7.34 -> 0.00 mm
- net SPI1_MISO: track 0.00 -> 4.48 mm
- net SPI1_CLK: track 0.00 -> 4.44 mm
- net SPI1_MOSI: track 0.00 -> 4.40 mm
- net /CLKN: track 7.34 -> 11.7 mm, vias 0 -> 2
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
Commit message: more stuff
Parts:
- removed ? (x3): , Graphics
- moved C7 75.4 mm to (118.7, 92.5), turned to 90 degrees
- moved C6 73.8 mm to (116.7, 92.5), turned to 90 degrees
- moved C5 72.4 mm to (114.7, 92.5), turned to 90 degrees
- moved C12 72.3 mm to (116.7, 83.7)
- moved C13 72.0 mm to (118.8, 80.5)
- moved C15 71.5 mm to (118.8, 78.5)
- moved C16 71.5 mm to (118.8, 79.5)
- moved C4 70.9 mm to (112.8, 92.5), turned to 90 degrees
- moved C3 69.6 mm to (110.8, 92.5), turned to 90 degrees
- moved R8 60.8 mm to (119.2, 77.0), turned to 90 degrees
- moved C8 60.7 mm to (105.0, 78.5), turned to 180 degrees
- moved R7 59.7 mm to (118.2, 77.0), turned to -90 degrees
- moved D1 58.3 mm to (116.0, 88.0), turned to 180 degrees
- moved C14 58.0 mm to (105.2, 74.7), turned to 180 degrees
- moved R10 58.0 mm to (116.5, 86.5)
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- gave numbers to parts that had none: 3
Routing:
- net /CLKN: track 11.7 -> 0.00 mm, vias 2 -> 0
- net SDC0_D2/JTAG_TCK: track 8.57 -> 0.00 mm
- net SDC0_D3: track 8.53 -> 0.00 mm
- net SDC0_CMD/JTAG_TDO: track 8.49 -> 0.00 mm
- net SDC0_CLK: track 8.45 -> 0.00 mm
- net SDC0_D0/JTAG_TDI: track 8.40 -> 0.00 mm
- net SDC0_D1/JTAG_TMS: track 8.36 -> 0.00 mm
- net /CLKP: track 6.73 -> 0.00 mm
- net SPI1_MISO: track 4.48 -> 0.00 mm
- net SPI1_CLK: track 4.44 -> 0.00 mm
- net SPI1_MOSI: track 4.40 -> 0.00 mm
- net SPI1_CS: track 4.36 -> 0.00 mm
- net +2V6: track 9.84 -> 6.91 mm
- net +3V3: track 9.96 -> 7.76 mm
- net +1V1: track 8.01 -> 6.54 mm

Commit message: stuff
Parts:
- moved J5 52.3 mm to (69.3, 82.9)
- moved U6 45.4 mm to (57.0, 80.5), turned to 90 degrees
- moved R9 40.7 mm to (55.6, 85.7), turned to 0 degrees
- moved Y1 23.9 mm to (103.9, 87.7), turned to -45 degrees
- moved C17 23.3 mm to (106.0, 89.3), turned to -135 degrees
- moved C18 22.4 mm to (101.8, 86.1), turned to 45 degrees
- moved SW1 19.1 mm to (118.0, 90.2), turned to -45 degrees
- moved C4 17.9 mm to (114.0, 74.6), turned to 45 degrees
- moved R12 17.3 mm to (115.8, 87.0), turned to 135 degrees
- moved D1 17.1 mm to (113.3, 71.1), turned to -135 degrees
- moved R10 16.5 mm to (115.4, 70.0), turned to 135 degrees
- moved C14 16.4 mm to (114.4, 88.3), turned to -45 degrees
- moved C3 15.5 mm to (118.1, 78.8), turned to 45 degrees
- moved R8 14.8 mm to (104.6, 79.1), turned to -45 degrees
- moved Q2 14.2 mm to (115.9, 72.4), turned to 135 degrees
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Routing:
- net +3V3: track 7.76 -> 19.6 mm
- net /CLKN: track 0.00 -> 8.51 mm
- net +2V6: track 6.91 -> 15.2 mm
- net Net-(U4B-SVREF): track 0.00 -> 6.51 mm, vias 0 -> 2
- net ~{RESET}: track 0.00 -> 6.49 mm, vias 0 -> 2
- net /CLKP: track 0.00 -> 5.93 mm
- net STATUS: track 0.00 -> 5.07 mm
- net +1V1: track 6.54 -> 10.6 mm
- net Net-(Q2-D): track 0.00 -> 1.84 mm
- net SPI_CS: track 0.00 -> 1.66 mm
- net Net-(D1-K): track 0.00 -> 1.52 mm

Commit message: full pbc layout completed
Parts:
- moved U6 57.7 mm to (112.5, 96.2), turned to 0 degrees
- moved R9 55.3 mm to (110.5, 92.7)
- moved J5 31.6 mm to (100.9, 82.8), turned to -135 degrees
- moved R8 1.41 mm to (103.5, 78.2), turned to 135 degrees
- moved C6 0.46 mm to (112.8, 89.5)
Routing:
- net GND: track 0.00 -> 253.3 mm, vias 0 -> 11
- net +3V3: track 19.6 -> 121.0 mm, vias 1 -> 10
- net +2V6: track 15.2 -> 66.8 mm, vias 1 -> 5
- net +1V1: track 10.6 -> 59.6 mm, vias 1 -> 6
- net +5V: track 24.2 -> 65.5 mm, vias 1 -> 3
- net SDC0_D2/JTAG_TCK: track 0.00 -> 41.0 mm, vias 0 -> 2
- net SDC0_D3: track 0.00 -> 37.8 mm, vias 0 -> 2
- net MICIN: track 0.00 -> 37.0 mm
- net SDC0_CLK: track 0.00 -> 36.4 mm, vias 0 -> 2
- net HPR: track 0.00 -> 34.2 mm
- net HPL: track 0.00 -> 32.7 mm, vias 0 -> 2
- net SDC0_CMD/JTAG_TDO: track 0.00 -> 31.6 mm, vias 0 -> 2
- net SDC0_D1/JTAG_TMS: track 0.00 -> 30.3 mm, vias 0 -> 2
- net SDC0_D0/JTAG_TDI: track 0.00 -> 26.6 mm, vias 0 -> 2
- net SCL: track 0.00 -> 24.1 mm, vias 0 -> 2
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- removed copper zone on In3.Cu, net GND
- removed copper zone on In4.Cu, net GND
Other:
- copper layers 6 -> 4
- board text added: "Layout by Εδέμ"

Commit message: h
Parts:
- added G***: LOGO, LOGO, F.Cu at (124.5, 102.2)
- added G***: LOGO, LOGO, F.Cu at (129.5, 104.0)
- added G***: LOGO, LOGO, F.Cu at (128.7, 100.8)
- added G***: LOGO, LOGO, F.Cu at (135.0, 98.5)
- added G***: LOGO, LOGO, F.Cu at (134.8, 103.5)
- added REF**: OSHW-Symbol_6.7x6mm_Copper, Symbol:OSHW-Symbol_6.7x6mm_Copper, F.Cu at (125.8, 106.2)
Routing:
- net D-: track 22.2 -> 21.5 mm
- net D+: track 22.3 -> 21.7 mm
Other:
- board text removed: "Layout by Εδέμ"
